File: power-supply.sch (KiCad schematic (older format))
At the start: 15 parts

Commit message: Wyprowadzenie VDD (3,3V); komentarze
Parts:
- added D?: D, symbol D
- added D?: 3,3V, symbol ZENER
- added R?: 220, symbol R
Connections:
- net labels added: 200VGND, 5VDC, VDD
- net labels removed: +5V, 200VGND?
- wire segments 42 -> 46
Other:
- note added: "TODO - scalak?"
- note added: "Zabezpieczenie\nukładu 7805"
- moved on the sheet: C?, D?, U?
Changed lines of the file:
@@
 L LM7805 U?
 U 1 1 581516AA
-P 7700 2000
-F 0 "U?" H 7850 1804 50  0000 C CNN
-F 1 "LM7805" H 7700 2200 50  0000 C CNN
-F 2 "" H 7700 2000 50  0000 C CNN
-F 3 "" H 7700 2000 50  0000 C CNN
-	1    7700 2000
+P 7150 2500
+F 0 "U?" H 7300 2304 50  0000 C CNN
+F 1 "LM7805" H 7150 2700 50  0000 C CNN
+F 2 "" H 7150 2500 50  0000 C CNN
+F 3 "" H 7150 2500 50  0000 C CNN
+	1    7150 2500
 	1    0    0    -1
 $EndComp
@@
 L CP C?
 U 1 1 58151831
-P 6550 2250
-F 0 "C?" H 6575 2350 50  0000 L CNN
-F 1 "4000u?" H 6575 2150 50  0000 L CNN
-F 2 "" H 6588 2100 50  0000 C CNN
-F 3 "" H 6550 2250 50  0000 C CNN
-	1    6550 2250
+P 6000 2750
+F 0 "C?" H 6025 2850 50  0000 L CNN
+F 1 "4000u?" H 6025 2650 50  0000 L CNN
+F 2 "" H 6038 2600 50  0000 C CNN
+F 3 "" H 6000 2750 50  0000 C CNN
+	1    6000 2750
 	1    0    0    -1
 $EndComp
@@
 L CP C?
 U 1 1 581518E5
-P 8800 2250
-F 0 "C?" H 8825 2350 50  0000 L CNN
-F 1 "400u?" H 8825 2150 50  0000 L CNN
-F 2 "" H 8838 2100 50  0000 C CNN
-F 3 "" H 8800 2250 50  0000 C CNN
-	1    8800 2250
+P 8250 2750
+F 0 "C?" H 8275 2850 50  0000 L CNN
+F 1 "400u?" H 8275 2650 50  0000 L CNN
+F 2 "" H 8288 2600 50  0000 C CNN
+F 3 "" H 8250 2750 50  0000 C CNN
+	1    8250 2750
 	1    0    0    -1
 $EndComp
@@
 L C C?
 U 1 1 58151B4F
-P 7150 2250
-F 0 "C?" H 7175 2350 50  0000 L CNN
-F 1 "1u" H 7175 2150 50  0000 L CNN
-F 2 "" H 7188 2100 50  0000 C CNN
-F 3 "" H 7150 2250 50  0000 C CNN
-	1    7150 2250
+P 6600 2750
+F 0 "C?" H 6625 2850 50  0000 L CNN
+F 1 "1u" H 6625 2650 50  0000 L CNN
+F 2 "" H 6638 2600 50  0000 C CNN
+F 3 "" H 6600 2750 50  0000 C CNN
+	1    6600 2750
 	1    0    0    -1
 $EndComp
@@
 L C C?
 U 1 1 58151BB1
-P 8200 2250
-F 0 "C?" H 8225 2350 50  0000 L CNN
-F 1 "1u" H 8225 2150 50  0000 L CNN
-F 2 "" H 8238 2100 50  0000 C CNN
-F 3 "" H 8200 2250 50  0000 C CNN
-	1    8200 2250
-	1    0    0    -1
-$EndComp
-Wire Wire Line
-	7150 1600 7150 2100
-Wire Wire Line
-	5300 1950 7300 1950
-Wire Wire Line
-	6550 2100 6550 1950
-Connection ~ 7150 1950
-Wire Wire Line
-	8100 1950 9450 1950
-Wire Wire Line
-	8200 1600 8200 2100
-Wire Wire Line
-	8800 1950 8800 2100
-Connection ~ 8200 1950
-Connection ~ 8800 1950
-Wire Wire Line
-	6550 2400 6550 2600
-Wire Wire Line
-	5500 2600 9450 2600
-Wire Wire Line
-	7700 2250 7700 2600
-Connection ~ 7700 2600
-Wire Wire Line
-	8800 2600 8800 2400
-Connection ~ 8800 2600
-Wire Wire Line
-	7150 2400 7250 2500
-Wire Wire Line
-	7250 2500 8100 2500
-Connection ~ 7700 2500
-Wire Wire Line
-	8100 2500 8200 2400
-Wire Wire Line
-	5300 1950 5300 4400
-Connection ~ 6550 1950
-Wire Wire Line
-	5500 2600 5500 5450
-Connection ~ 6550 2600
-$Comp
-L GND #PWR?
-U 1 1 58152CDA
-P 9450 2650
-F 0 "#PWR?" H 9450 2400 50  0001 C CNN
-F 1 "GND" H 9450 2500 50  0000 C CNN
-F 2 "" H 9450 2650 50  0000 C CNN
-F 3 "" H 9450 2650 50  0000 C CNN
-	1    9450 2650
-	1    0    0    -1
-$EndComp
-Wire Wire Line
-	9450 2600 9450 2650
-$Comp
-L +5V #PWR?
-U 1 1 58152D37
-P 9450 1900
-F 0 "#PWR?" H 9450 1750 50  0001 C CNN
-F 1 "+5V" H 9450 2040 50  0000 C CNN
-F 2 "" H 9450 1900 50  0000 C CNN
-F 3 "" H 9450 1900 50  0000 C CNN
-	1    9450 1900
-	1    0    0    -1
-$EndComp
-Wire Wire Line
-	9450 1950 9450 1900
+P 7650 2750
+F 0 "C?" H 7675 2850 50  0000 L CNN
+F 1 "1u" H 7675 2650 50  0000 L CNN
+F 2 "" H 7688 2600 50  0000 C CNN
+F 3 "" H 7650 2750 50  0000 C CNN
+	1    7650 2750
+	1    0    0    -1
+$EndComp
+Wire Wire Line
+	6600 2100 6600 2600
+Wire Wire Line
+	5300 2450 6750 2450
+Wire Wire Line
+	6000 2600 6000 2450
+Connection ~ 6600 2450
+Wire Wire Line
+	7550 2450 9450 2450
+Wire Wire Line
+	7650 2100 7650 2600
+Wire Wire Line
+	8250 2450 8250 2600
+Connection ~ 7650 2450
+Connection ~ 8250 2450
+Wire Wire Line
+	6000 2900 6000 3100
+Wire Wire Line
+	5500 3100 9450 3100
+Wire Wire Line
+	7150 2750 7150 3100
+Connection ~ 7150 3100
+Wire Wire Line
+	8250 3100 8250 2900
+Connection ~ 8250 3100
+Wire Wire Line
+	6600 2900 6700 3000
+Wire Wire Line
+	6700 3000 7550 3000
+Connection ~ 7150 3000
+Wire Wire Line
+	7550 3000 7650 2900
+Wire Wire Line
+	5300 2450 5300 4400
+Connection ~ 6000 2450
+Wire Wire Line
+	5500 3100 5500 5450
+Connection ~ 6000 3100
 $Comp
 L INDUCTOR L?
@@
 L D D?
 U 1 1 581539A7
-P 7700 1600
-F 0 "D?" H 7700 1700 50  0000 C CNN
-F 1 "D" H 7700 1500 50  0000 C CNN
-F 2 "" H 7700 1600 50  0000 C CNN
-F 3 "" H 7700 1600 50  0000 C CNN
-	1    7700 1600
-	1    0    0    -1
-$EndComp
-Wire Wire Line
-	7850 1600 8200 1600
-Wire Wire Line
-	7550 1600 7150 1600
+P 7150 2100
+F 0 "D?" H 7150 2200 50  0000 C CNN
+F 1 "D" H 7150 2000 50  0000 C CNN
+F 2 "" H 7150 2100 50  0000 C CNN
+F 3 "" H 7150 2100 50  0000 C CNN
+	1    7150 2100
+	1    0    0    -1
+$EndComp
+Wire Wire Line
+	7300 2100 7650 2100
+Wire Wire Line
+	7000 2100 6600 2100
 $Comp
 L Q_NMOS_DGS Q?
@@
 Connection ~ 7250 4400
 Wire Wire Line
-	7850 4400 9050 4400
+	7850 4400 9450 4400
 Wire Wire Line
 	8300 4400 8300 4700
 Connection ~ 8300 4400
-Wire Wire Line
-	5300 4400 6400 4400
 Connection ~ 5300 3500
 Wire Wire Line
 	7250 5050 7250 5450
 Wire Wire Line
-	5500 5450 9050 5450
+	5500 5450 9450 5450
 Wire Wire Line
 	8300 5450 8300 5000
@@
 Connection ~ 7250 5450
 Connection ~ 5500 3900
-Text Label 8700 4400 0    60   ~ 0
-200VDC
-Text Label 8650 5450 0    60   ~ 0
-200VGND?
 Wire Wire Line
 	6250 4850 6950 4850
 Text Label 6250 4850 0    60   ~ 0
 PWM_BRIGHT
+$Comp
+L D D?
+U 1 1 58170BE4
+P 5950 4400
+F 0 "D?" H 5950 4500 50  0000 C CNN
+F 1 "D" H 5950 4300 50  0000 C CNN
+F 2 "" H 5950 4400 50  0000 C CNN
+F 3 "" H 5950 4400 50  0000 C CNN
+	1    5950 4400
+	-1   0    0    1
+$EndComp
+Wire Wire Line
+	5300 4400 5800 4400
+Wire Wire Line
+	6100 4400 6400 4400
+Text Notes 6250 4200 2    60   ~ 0
+Zabezpieczenie\nukładu 7805
+Text HLabel 9450 1600 2    60   Output ~ 0
+VDD
+Text HLabel 9450 3100 2    60   Output ~ 0
+GND
+Text HLabel 9450 4400 2    60   Output ~ 0
+200VDC
+Text HLabel 9450 5450 2    60   Output ~ 0
+200VGND
+$Comp
+L ZENER D?
+U 1 1 58179AB5
+P 9150 1950
+F 0 "D?" H 9150 2050 50  0000 C CNN
+F 1 "3,3V" H 9150 1850 50  0000 C CNN
+F 2 "" H 9150 1950 50  0000 C CNN
+F 3 "" H 9150 1950 50  0000 C CNN
+F 4 "1N5913B" H 9150 1950 60  0001 C CNN "Part no."
+	1    9150 1950
+	0    1    1    0
+$EndComp
+$Comp
+L R R?
+U 1 1 58179BE8
+P 8750 1600
+F 0 "R?" V 8830 1600 50  0000 C CNN
+F 1 "220" V 8750 1600 50  0000 C CNN
+F 2 "" V 8680 1600 50  0000 C CNN
+F 3 "" H 8750 1600 50  0000 C CNN
+	1    8750 1600
+	0    1    1    0
+$EndComp
+Wire Wire Line
+	8450 2450 8450 1600
+Wire Wire Line
+	8450 1600 8600 1600
+Connection ~ 8450 2450
+Wire Wire Line
+	8900 1600 9450 1600
+Wire Wire Line
+	9150 1600 9150 1750
+Connection ~ 9150 1600
+Wire Wire Line
+	9150 2150 9150 3100
+Connection ~ 9150 3100
+Text HLabel 9450 2450 2    60   Output ~ 0
+5VDC
+Text Notes 9300 1450 2    60   ~ 0
+TODO - scalak?
 $EndSCHEMATC

Commit message: Kontrola jasnosci NIXIE
Connections:
- net PWM_BRIGHT renamed BRIGHT_PWM
Changed lines of the file:
@@
 Connection ~ 5500 3900
 Wire Wire Line
-	6250 4850 6950 4850
-Text Label 6250 4850 0    60   ~ 0
-PWM_BRIGHT
+	1250 4850 6950 4850
 $Comp
 L D D?
@@
 Text Notes 9300 1450 2    60   ~ 0
 TODO - scalak?
+Text HLabel 1250 4850 0    60   Input ~ 0
+BRIGHT_PWM
 $EndSCHEMATC
