File: nixie-module/nixie-module.kicad_pcb (KiCad board)
At the start: 2 copper layers, 5 parts, among them P1 CONN_02X05, U1 74141

Commit message: Poprawki; otwory montazowe; obrys
Parts:
- added REF**: MountingHole_3.2mm_M3, Mounting_Holes:MountingHole_3.2mm_M3, F.Cu at (160.0, 124.2)
- added REF**: MountingHole_3.2mm_M3, Mounting_Holes:MountingHole_3.2mm_M3, F.Cu at (132.0, 76.2)
Routing:
- net Net-(E1-Pad11): track 40.1 -> 37.3 mm
- net Net-(E1-Pad5): track 50.0 -> 52.5 mm
- net Net-(E1-Pad4): track 47.4 -> 49.0 mm
- net VCC: track 64.3 -> 65.6 mm
- net Net-(E1-Pad12): track 47.2 -> 46.3 mm
- net Net-(E1-Pad9): track 9.58 -> 10.1 mm
Other:
- board outline added: 36 x 56 mm
