File: main-board/nixie-clock.kicad_pcb (KiCad board)
At the start: 2 copper layers, 168.7 x 41.1 mm, 57 parts, among them P1 ESP8266_CONN, P2 CONN_01X06, P3 CONN_01X03, P4 CONN_02X05, P5 CONN_02X05, P6 CONN_02X05, P7 CONN_02X05, Q1 2N7002, Q2 2N7002, Q3 BSP324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

Commit message: wygenerowanie plików produkcyjnych do płytki main-board
Routing:
- net GND: track 90.0 -> 87.5 mm, vias 16 -> 15
- net (no net): track 0.00 -> 2.54 mm, vias 0 -> 1
Changed lines of the file:
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@@
     (visible_elements 7FFEFFFF)
     (pcbplotparams
-      (layerselection 0x00030_80000001)
-      (usegerberextensions false)
+      (layerselection 0x010f0_ffffffff)
+      (usegerberextensions true)
       (excludeedgelayer true)
       (linewidth 0.100000)
@@
       (psa4output false)
       (plotreference true)
-      (plotvalue true)
+      (plotvalue false)
       (plotinvisibletext false)
       (padsonsilk false)
@@
       (outputformat 1)
       (mirror false)
-      (drillshape 1)
+      (drillshape 0)
       (scaleselection 1)
-      (outputdirectory ""))
+      (outputdirectory gerber/))
   )
   (net 0 "")
@@
     (arrow2b (pts (xy 171.45 156.21) (xy 172.576504 155.623579)))
   )
-  (segment (start 126.492 136.2075) (end 127.8255 136.2075) (width 0.3048) (layer B.Cu) (net 1))
-  (segment (start 127.8255 136.2075) (end 129.032 136.2075) (width 0.3048) (layer F.Cu) (net 1))
-  (via (at 127.8255 136.2075) (size 0.889) (drill 0.635) (layers F.Cu B.Cu) (net 1))
+  (segment (start 126.492 136.2075) (end 127.8255 136.2075) (width 0.3048) (layer B.Cu) (net 0))
+  (segment (start 127.8255 136.2075) (end 129.032 136.2075) (width 0.3048) (layer F.Cu) (net 0))
+  (via (at 127.8255 136.2075) (size 0.889) (drill 0.635) (layers F.Cu B.Cu) (net 0))
   (segment (start 145.1236 131.6294) (end 145.1236 133.3888) (width 0.254) (layer F.Cu) (net 1))
   (segment (start 146.276928 134.542128) (end 146.177 134.4422) (width 0.254) (layer F.Cu) (net 1))
@@
   (segment (start 161.2265 131.9022) (end 161.2265 131.6355) (width 1.524) (layer F.Cu) (net 39))
   (segment (start 159.1183 133.4135) (end 149.9035 133.4135) (width 1.524) (layer F.Cu) (net 39))
-  (segment (start 149.9035 133.4135) (end 149.6876 133.6294) (width 1.524) (layer F.Cu) (net 39) (status C00000))
+  (segment (start 149.9035 133.4135) (end 149.6876 133.6294) (width 1.524) (layer F.Cu) (net 39))
   (segment (start 170.8658 124.253) (end 167.814 124.253) (width 0.381) (layer F.Cu) (net 39))
   (segment (start 167.814 124.253) (end 166.2938 122.7328) (width 0.381) (layer F.Cu) (net 39))
@@
   (segment (start 158.8516 122.98934) (end 158.09214 123.7488) (width 1.524) (layer F.Cu) (net 39))
   (segment (start 158.09214 123.7488) (end 156.14904 123.7488) (width 1.524) (layer F.Cu) (net 39))
-  (segment (start 166.2938 122.7328) (end 161.48812 121.9708) (width 1.524) (layer F.Cu) (net 39) (status 400000))
+  (segment (start 166.2938 122.7328) (end 161.48812 121.9708) (width 1.524) (layer F.Cu) (net 39))
   (segment (start 161.48812 121.9708) (end 161.23158 122.22734) (width 1.524) (layer F.Cu) (net 39))
-  (segment (start 161.23158 122.22734) (end 158.8516 122.98934) (width 1.524) (layer F.Cu) (net 39) (status 800000))
+  (segment (start 161.23158 122.22734) (end 158.8516 122.98934) (width 1.524) (layer F.Cu) (net 39))
   (segment (start 62.3316 126.4666) (end 62.332 128.7526) (width 1.524) (layer F.Cu) (net 39))
   (segment (start 62.332 128.7526) (end 62.68466 129.10526) (width 1.524) (layer F.Cu) (net 39))
@@
   (segment (start 158.5595 128.5875) (end 158.5595 128.7145) (width 0.381) (layer B.Cu) (net 46))
   (segment (start 183.007 132.461) (end 183.1175 132.3505) (width 0.381) (layer B.Cu) (net 46))
-  (segment (start 183.1175 132.3505) (end 184.0865 132.3505) (width 0.381) (layer B.Cu) (net 46) (status 800000))
+  (segment (start 183.1175 132.3505) (end 184.0865 132.3505) (width 0.381) (layer B.Cu) (net 46))
   (segment (start 181.6735 133.7945) (end 183.7055 133.7945) (width 0.381) (layer F.Cu) (net 46))
   (via (at 181.6735 133.7945) (size 0.889) (drill 0.635) (layers F.Cu B.Cu) (net 46))
